Commit message: -

File: basic_robot_description/urdf/basic_robot.xacro (robot description, xacro)
@@ -2,5 +2,5 @@
 <robot name="basic_robot" xmlns:xacro="http://www.ros.org/wiki/xacro">
 <xacro:include filename="$(find basic_robot_description)/urdf/materials.xacro" />
-<xacro:include filename="$(find basic_robot_description)/urdf/basic_robot.trans" />
+<xacro:include filename="$(find basic_robot_description)/urdf/basic_robot.ros2control" />
 <xacro:include filename="$(find basic_robot_description)/urdf/basic_robot.gazebo" />
 <link name="base_link">
@@ -13,5 +13,5 @@
     <origin xyz="0 0 0" rpy="0 0 0"/>
     <geometry>
-      <mesh filename="package://basic_robot_description/meshes/base_link.stl" scale="0.001 0.001 0.001"/>
+      <mesh filename="file://$(find basic_robot_description)/meshes/base_link.stl" scale="0.001 0.001 0.001"/>
     </geometry>
     <material name="silver"/>
@@ -20,109 +20,7 @@
     <origin xyz="0 0 0" rpy="0 0 0"/>
     <geometry>
-      <mesh filename="package://basic_robot_description/meshes/base_link.stl" scale="0.001 0.001 0.001"/>
+      <mesh filename="file://$(find basic_robot_description)/meshes/base_link.stl" scale="0.001 0.001 0.001"/>
     </geometry>
   </collision>
 </link>
-<link name="right_wheel_link_1">
-  <inertial>
-    <origin xyz="-0.004968790442628317 2.6645352591003757e-15 0.0" rpy="0 0 0"/>
-    <mass value="0.01795474341761617"/>
-    <inertia ixx="6e-06" iyy="3e-06" izz="3e-06" ixy="0.0" iyz="0.0" ixz="0.0"/>
-  </inertial>
-  <visual>
-    <origin xyz="0.045 -0.045 -0.025" rpy="0 0 0"/>
-    <geometry>
-      <mesh filename="package://basic_robot_description/meshes/right_wheel_link_1.stl" scale="0.001 0.001 0.001"/>
-    </geometry>
-    <material name="silver"/>
-  </visual>
-  <collision>
-    <origin xyz="0.045 -0.045 -0.025" rpy="0 0 0"/>
-    <geometry>
-      <mesh filename="package://basic_robot_description/meshes/right_wheel_link_1.stl" scale="0.001 0.001 0.001"/>
-    </geometry>
-  </collision>
-</link>
-<link name="left_wheel_link_1">
-  <inertial>
-    <origin xyz="0.00496879044262831 2.67841304690819e-15 3.469446951953614e-18" rpy="0 0 0"/>
-    <mass value="0.017954743417616166"/>
-    <inertia ixx="6e-06" iyy="3e-06" izz="3e-06" ixy="0.0" iyz="0.0" ixz="0.0"/>
-  </inertial>
-  <visual>
-    <origin xyz="-0.045 -0.045 -0.025" rpy="0 0 0"/>
-    <geometry>
-      <mesh filename="package://basic_robot_description/meshes/left_wheel_link_1.stl" scale="0.001 0.001 0.001"/>
-    </geometry>
-    <material name="silver"/>
-  </visual>
-  <collision>
-    <origin xyz="-0.045 -0.045 -0.025" rpy="0 0 0"/>
-    <geometry>
-      <mesh filename="package://basic_robot_description/meshes/left_wheel_link_1.stl" scale="0.001 0.001 0.001"/>
-    </geometry>
-  </collision>
-</link>
-<link name="lidar_1">
-  <inertial>
-    <origin xyz="0.0 6.938893903907228e-18 0.00508531611148879" rpy="0 0 0"/>
-    <mass value="0.09858736625985248"/>
-    <inertia ixx="1e-05" iyy="1e-05" izz="1.9e-05" ixy="0.0" iyz="0.0" ixz="0.0"/>
-  </inertial>
-  <visual>
-    <origin xyz="-0.0 -0.03 -0.05" rpy="0 0 0"/>
-    <geometry>
-      <mesh filename="package://basic_robot_description/meshes/lidar_1.stl" scale="0.001 0.001 0.001"/>
-    </geometry>
-    <material name="silver"/>
-  </visual>
-  <collision>
-    <origin xyz="-0.0 -0.03 -0.05" rpy="0 0 0"/>
-    <geometry>
-      <mesh filename="package://basic_robot_description/meshes/lidar_1.stl" scale="0.001 0.001 0.001"/>
-    </geometry>
-  </collision>
-</link>
-<link name="caster_link_1">
-  <inertial>
-    <origin xyz="2.5130308594279645e-18 0.020000000000000004 -0.005625000000000003" rpy="0 0 0"/>
-    <mass value="0.056548667764616256"/>
-    <inertia ixx="3e-06" iyy="3e-06" izz="5e-06" ixy="0.0" iyz="0.0" ixz="-0.0"/>
-  </inertial>
-  <visual>
-    <origin xyz="-0.0 0.06 -0.015" rpy="0 0 0"/>
-    <geometry>
-      <mesh filename="package://basic_robot_description/meshes/caster_link_1.stl" scale="0.001 0.001 0.001"/>
-    </geometry>
-    <material name="silver"/>
-  </visual>
-  <collision>
-    <origin xyz="-0.0 0.06 -0.015" rpy="0 0 0"/>
-    <geometry>
-      <mesh filename="package://basic_robot_description/meshes/caster_link_1.stl" scale="0.001 0.001 0.001"/>
-    </geometry>
-  </collision>
-</link>
-<joint name="Revolute 1" type="continuous">
-  <origin xyz="-0.045 0.045 0.025" rpy="0 0 0"/>
-  <parent link="base_link"/>
-  <child link="right_wheel_link_1"/>
-  <axis xyz="-1.0 0.0 0.0"/>
-</joint>
-<joint name="Revolute 2" type="continuous">
-  <origin xyz="0.045 0.045 0.025" rpy="0 0 0"/>
-  <parent link="base_link"/>
-  <child link="left_wheel_link_1"/>
-  <axis xyz="1.0 0.0 0.0"/>
-</joint>
-<joint name="Rigid 3" type="fixed">
-  <origin xyz="0.0 0.03 0.05" rpy="0 0 0"/>
-  <parent link="base_link"/>
-  <child link="lidar_1"/>
-</joint>
-<joint name="Rigid 4" type="fixed">
-  <origin xyz="0.0 -0.06 0.015" rpy="0 0 0"/>
-  <parent link="base_link"/>
-  <child link="caster_link_1"/>
-</joint>
 </robot>
